File: Relay_Driver_4_motor/Relay_Driver.kicad_pcb (KiCad board)
At the start: 2 copper layers, 38 parts, among them J1 Conn_01x10, M1 Conn_01x02, M2 Conn_01x02, M3 Conn_01x02, M4 Conn_01x02, SW1 SW_SPDT, SW2 SW_SPDT, U1 ULN2803A

Commit message: completed routing
Parts:
- J1: footprint Pin_Headers:Pin_Header_Straight_1x10_Pitch1.00mm -> Pin_Headers:Pin_Header_Straight_1x10_Pitch2.54mm
- RL1M1, RL1M2, RL1M3, RL1M4, RL2M1, RL2M2, RL2M3, RL2M4: footprint Relays_THT:Relay_SPDT_OMRON-G5LE-1 -> Relay_Driver_4_motor_modded:Relay_SPDT_OMRON-G5LE-1
- SW1, SW2: footprint Buttons_Switches_THT:SW_CuK_OS102011MA1QN1_SPDT_Angled -> Connectors_WAGO:WAGO_734_3pin_Straight
- moved D9 140.4 mm to (79.2, 163.1), turned to 180 degrees
- moved D10 129.6 mm to (66.5, 138.4), turned to 0 degrees
- moved RL1M4 124.1 mm to (65.1, 151.0), turned to 90 degrees
- moved M4 113.6 mm to (48.5, 138.7), turned to 270 degrees
- moved D2 104.4 mm to (111.8, 163.1), turned to 180 degrees
- moved RL2M4 90.3 mm to (65.1, 120.0), turned to 90 degrees
- moved SW2 88.7 mm to (53.6, 153.4), turned to 180 degrees
- moved D15 87.7 mm to (79.2, 132.3), turned to 180 degrees
- moved RL1M3 85.6 mm to (113.3, 151.0), turned to 270 degrees
- moved D7 82.5 mm to (99.1, 138.4), turned to 0 degrees
- moved D14 77.6 mm to (99.1, 47.0), turned to 0 degrees
- moved C1 76.4 mm to (50.3, 127.5), turned to 270 degrees
- moved M1 74.8 mm to (47.8, 81.1), turned to 90 degrees
- moved D16 73.2 mm to (66.5, 107.2), turned to 0 degrees
- moved D12 72.3 mm to (111.8, 100.8), turned to 180 degrees
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Routing:
- net +5V: track 0.00 -> 598.2 mm
- net GND: track 0.00 -> 577.1 mm
- net +12V: track 0.00 -> 335.0 mm
- net Net-(RL1M2-Pad1): track 0.00 -> 172.6 mm
- net Net-(RL2M3-Pad1): track 0.00 -> 160.8 mm
- net Net-(RL1M3-Pad1): track 0.00 -> 140.1 mm
- net Net-(RL2M2-Pad1): track 0.00 -> 135.8 mm
- net Net-(RL1M4-Pad1): track 0.00 -> 75.6 mm
- net Net-(D1-Pad2): track 0.00 -> 70.3 mm
- net Net-(RL2M1-Pad1): track 0.00 -> 67.1 mm
- net Net-(D5-Pad1): track 0.00 -> 52.2 mm
- net Net-(D15-Pad2): track 0.00 -> 50.8 mm
- net Net-(D10-Pad1): track 0.00 -> 47.8 mm
- net Net-(C1-Pad1): track 0.00 -> 46.6 mm
- net Net-(D11-Pad2): track 0.00 -> 40.5 mm
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- added copper zone on B.Cu, net GND
